Commit message: update

File: turtlebot3_description/urdf/turtlebot3_waffle_pi.urdf.xacro (robot description, xacro)
@@ -173,4 +173,5 @@
     </collision>
   </link>
+<!--center-->
   <joint name="camera_rgb_joint" type="fixed">
     <origin xyz="0.003 0.011 0.009" rpy="0 0 0"/>
@@ -185,6 +186,34 @@
   </joint>
   <link name="camera_rgb_optical_frame"/>
+<!--center_left-->
+  <joint name="camera_rgb_center_left_joint" type="fixed">
+    <origin xyz="0.003 0.011 0.009" rpy="0 0 0.088"/>
+    <parent link="camera_link"/>
+    <child link="camera_rgb_center_left_frame"/>
+  </joint>
+  <link name="camera_rgb_center_left_frame"/>
+  <joint name="camera_rgb_optical_center_left_joint" type="fixed">
+    <origin xyz="0 0 0" rpy="-1.57 0 -1.57"/>
+    <parent link="camera_rgb_center_left_frame"/>
+    <child link="camera_rgb_optical_center_left_frame"/>
+  </joint>
+  <link name="camera_rgb_optical_center_left_frame"/>
+<!--center_right-->
+  <joint name="camera_rgb_center_right_joint" type="fixed">
+    <origin xyz="0.003 0.011 0.009" rpy="0 0 -0.088"/>
+    <parent link="camera_link"/>
+    <child link="camera_rgb_center_right_frame"/>
+  </joint>
+  <link name="camera_rgb_center_right_frame"/>
+  <joint name="camera_rgb_optical_center_right_joint" type="fixed">
+    <origin xyz="0 0 0" rpy="-1.57 0 -1.57"/>
+    <parent link="camera_rgb_center_right_frame"/>
+    <child link="camera_rgb_optical_center_right_frame"/>
+  </joint>
+  <link name="camera_rgb_optical_center_right_frame"/>
+<!--left-->
   <joint name="camera_rgb_left_joint" type="fixed">
-    <origin xyz="0.003 0.111 0.009" rpy="0 0 0.175"/>
+    <!-- <origin xyz="0.003 0.111 0.009" rpy="0 0 0.175"/> -->
+     <origin xyz="0.003 0.211 0.009" rpy="0 0 0"/>
     <parent link="camera_link"/>
     <child link="camera_rgb_left_frame"/>
@@ -197,6 +226,34 @@
   </joint>
   <link name="camera_rgb_optical_left_frame"/>
+<!--left_left-->
+  <joint name="camera_rgb_left_left_joint" type="fixed">
+     <origin xyz="0.003 0.211 0.009" rpy="0 0 0.088"/>
+    <parent link="camera_link"/>
+    <child link="camera_rgb_left_left_frame"/>
+  </joint>
+  <link name="camera_rgb_left_left_frame"/>
+  <joint name="camera_rgb_optical_left_left_joint" type="fixed">
+    <origin xyz="0 0 0" rpy="-1.57 0 -1.57"/>
+    <parent link="camera_rgb_left_left_frame"/>
+    <child link="camera_rgb_optical_left_left_frame"/>
+  </joint>
+  <link name="camera_rgb_optical_left_left_frame"/>
+<!--left_right-->
+  <joint name="camera_rgb_left_right_joint" type="fixed">
+     <origin xyz="0.003 0.211 0.009" rpy="0 0 -0.088"/>
+    <parent link="camera_link"/>
+    <child link="camera_rgb_left_right_frame"/>
+  </joint>
+  <link name="camera_rgb_left_right_frame"/>
+  <joint name="camera_rgb_optical_left_right_joint" type="fixed">
+    <origin xyz="0 0 0" rpy="-1.57 0 -1.57"/>
+    <parent link="camera_rgb_left_right_frame"/>
+    <child link="camera_rgb_optical_left_right_frame"/>
+  </joint>
+  <link name="camera_rgb_optical_left_right_frame"/>
+<!--right-->
   <joint name="camera_rgb_right_joint" type="fixed">
-    <origin xyz="0.003 -0.089 0.009" rpy="0 0 -0.175"/>
+    <!-- <origin xyz="0.003 -0.089 0.009" rpy="0 0 -0.175"/> -->
+    <origin xyz="0.003 -0.189 0.009" rpy="0 0 0"/>
     <parent link="camera_link"/>
     <child link="camera_rgb_right_frame"/>
@@ -209,3 +266,29 @@
   </joint>
   <link name="camera_rgb_optical_right_frame"/>
+<!--right_left-->
+  <joint name="camera_rgb_right_left_joint" type="fixed">
+    <origin xyz="0.003 -0.189 0.009" rpy="0 0 0.088"/>
+    <parent link="camera_link"/>
+    <child link="camera_rgb_right_left_frame"/>
+  </joint>
+  <link name="camera_rgb_right_left_frame"/>
+  <joint name="camera_rgb_optical_right_left_joint" type="fixed">
+    <origin xyz="0 0 0" rpy="-1.57 0 -1.57"/>
+    <parent link="camera_rgb_right_left_frame"/>
+    <child link="camera_rgb_optical_right_left_frame"/>
+  </joint>
+  <link name="camera_rgb_optical_right_left_frame"/>
+<!--right_right-->
+  <joint name="camera_rgb_right_right_joint" type="fixed">
+    <origin xyz="0.003 -0.189 0.009" rpy="0 0 -0.088"/>
+    <parent link="camera_link"/>
+    <child link="camera_rgb_right_right_frame"/>
+  </joint>
+  <link name="camera_rgb_right_right_frame"/>
+  <joint name="camera_rgb_optical_right_right_joint" type="fixed">
+    <origin xyz="0 0 0" rpy="-1.57 0 -1.57"/>
+    <parent link="camera_rgb_right_right_frame"/>
+    <child link="camera_rgb_optical_right_right_frame"/>
+  </joint>
+  <link name="camera_rgb_optical_right_right_frame"/>
 </robot>
