Commit message: change urdf

File: turtlebot3_description/urdf/turtlebot3_waffle_pi.gazebo.xacro (robot description, xacro)
@@ -82,5 +82,5 @@
       <serviceName>imu_service</serviceName>
       <gaussianNoise>0.0</gaussianNoise>
-      <updateRate>200</updateRate>
+      <updateRate>0</updateRate>
       <imu>
         <noise>
@@ -118,6 +118,6 @@
         </scan>
         <range>
-          <min>0.120</min>
-          <max>3.5</max>
+          <min>0.2</min>
+          <max>30</max>
           <resolution>0.015</resolution>
         </range>
@@ -135,133 +135,11 @@
   </gazebo>
 <!--link : https://www.raspberrypi.org/documentation/hardware/camera/-->
-  <gazebo reference="camera_rgb_left_frame">
-    <sensor type="camera" name="camera_left">
+  <!-- <gazebo reference="camera_rgb_frame">
+    <sensor type="camera" name="Pi Camera">
       <always_on>true</always_on>
       <visualize>$(arg camera_visual)</visualize>
       <camera>
-          <!--120°-->
-          <horizontal_fov>2.09</horizontal_fov>
-          <!--130°-->
-          <!-- <horizontal_fov>2.27</horizontal_fov> -->
-          <!--150°-->
-          <!-- <horizontal_fov>2.62</horizontal_fov> -->
+          <horizontal_fov>1.085595</horizontal_fov>
           <image>
-              <!-- <width>694</width> -->
-              <!-- <height>520</height> -->
-              <width>640</width>
-              <height>480</height>
-              <format>R8G8B8</format>
-          </image>
-          <clip>
-              <near>0.03</near>
-              <far>100</far>
-          </clip>
-      </camera>
-      <plugin name="camera_controller" filename="libgazebo_ros_camera.so">
-		<topicName>camera_left</topicName>
-		<alwaysOn>true</alwaysOn>
-        <updateRate>30.0</updateRate>
-        <cameraName>camera_left</cameraName>
-        <frameName>camera_rgb_optical_left_frame</frameName>
-        <imageTopicName>rgb/image_raw</imageTopicName>
-        <cameraInfoTopicName>rgb/camera_info</cameraInfoTopicName>
-        <hackBaseline>0.07</hackBaseline>
-        <distortionK1>0.0</distortionK1>
-        <distortionK2>0.0</distortionK2>
-        <distortionK3>0.0</distortionK3>
-        <distortionT1>0.0</distortionT1>
-        <distortionT2>0.0</distortionT2>
-      </plugin>
-    </sensor>
-  </gazebo>
-<!--link : https://www.raspberrypi.org/documentation/hardware/camera/-->
-  <gazebo reference="camera_rgb_left_left_frame">
-    <sensor type="camera" name="camera_left_left">
-      <always_on>true</always_on>
-      <visualize>$(arg camera_visual)</visualize>
-      <camera>
-          <!--120°-->
-          <horizontal_fov>2.09</horizontal_fov>
-          <image>
-              <!-- <width>694</width>
-              <height>520</height> -->
-              <width>640</width>
-              <height>480</height>
-              <format>R8G8B8</format>
-          </image>
-          <clip>
-              <near>0.03</near>
-              <far>100</far>
-          </clip>
-      </camera>
-      <plugin name="camera_controller" filename="libgazebo_ros_camera.so">
-		<topicName>camera_left_left</topicName>
-		<alwaysOn>true</alwaysOn>
-        <updateRate>30.0</updateRate>
-        <cameraName>camera_left_left</cameraName>
-        <frameName>camera_rgb_optical_left_left_frame</frameName>
-        <imageTopicName>rgb/image_raw</imageTopicName>
-        <cameraInfoTopicName>rgb/camera_info</cameraInfoTopicName>
-        <hackBaseline>0.07</hackBaseline>
-        <distortionK1>0.0</distortionK1>
-        <distortionK2>0.0</distortionK2>
-        <distortionK3>0.0</distortionK3>
-        <distortionT1>0.0</distortionT1>
-        <distortionT2>0.0</distortionT2>
-      </plugin>
-    </sensor>
-  </gazebo>
-<!--link : https://www.raspberrypi.org/documentation/hardware/camera/-->
-  <gazebo reference="camera_rgb_left_right_frame">
-    <sensor type="camera" name="camera_left_right">
-      <always_on>true</always_on>
-      <visualize>$(arg camera_visual)</visualize>
-      <camera>
-          <!--120°-->
-          <horizontal_fov>2.09</horizontal_fov>
-          <image>
-              <!-- <width>694</width>
-              <height>520</height> -->
-              <width>640</width>
-              <height>480</height>
-              <format>R8G8B8</format>
-          </image>
-          <clip>
-              <near>0.03</near>
-              <far>100</far>
-          </clip>
-      </camera>
-      <plugin name="camera_controller" filename="libgazebo_ros_camera.so">
-		<topicName>camera_left_right</topicName>
-		<alwaysOn>true</alwaysOn>
-        <updateRate>30.0</updateRate>
-        <cameraName>camera_left_right</cameraName>
-        <frameName>camera_rgb_optical_left_right_frame</frameName>
-        <imageTopicName>rgb/image_raw</imageTopicName>
-        <cameraInfoTopicName>rgb/camera_info</cameraInfoTopicName>
-        <hackBaseline>0.07</hackBaseline>
-        <distortionK1>0.0</distortionK1>
-        <distortionK2>0.0</distortionK2>
-        <distortionK3>0.0</distortionK3>
-        <distortionT1>0.0</distortionT1>
-        <distortionT2>0.0</distortionT2>
-      </plugin>
-    </sensor>
-  </gazebo>
-<!--link : https://www.raspberrypi.org/documentation/hardware/camera/-->
-  <gazebo reference="camera_rgb_frame">
-    <sensor type="camera" name="camera">
-      <always_on>true</always_on>
-      <visualize>$(arg camera_visual)</visualize>
-      <camera>
-          <!--120°-->
-          <horizontal_fov>2.09</horizontal_fov>
-          <!--130°-->
-          <!-- <horizontal_fov>2.27</horizontal_fov> -->
-          <!--150°-->
-          <!-- <horizontal_fov>2.62</horizontal_fov> -->
-          <image>
-              <!-- <width>694</width> -->
-              <!-- <height>520</height> -->
               <width>640</width>
               <height>480</height>
@@ -288,33 +166,43 @@
       </plugin>
     </sensor>
-  </gazebo>
-<!--link : https://www.raspberrypi.org/documentation/hardware/camera/-->
-  <gazebo reference="camera_rgb_center_left_frame">
-    <sensor type="camera" name="camera_center_left">
-      <always_on>true</always_on>
-      <visualize>$(arg camera_visual)</visualize>
-      <camera>
-          <!--120°-->
-          <horizontal_fov>2.09</horizontal_fov>
+  </gazebo> -->
+  <gazebo reference="omnidirectional_camera_front_frame">
+      <sensor type="wideanglecamera" name="camera">
+        <camera>
+          <horizontal_fov>3.14</horizontal_fov>
           <image>
-              <!-- <width>694</width>
-              <height>520</height> -->
-              <width>640</width>
-              <height>480</height>
-              <format>R8G8B8</format>
+            <width>640</width>
+            <height>640</height>
           </image>
           <clip>
-              <near>0.03</near>
-              <far>100</far>
+            <near>0.1</near>
+            <far>50</far>
           </clip>
-      </camera>
-      <plugin name="camera_controller" filename="libgazebo_ros_camera.so">
+          <lens>
+            <!-- <type>gnomonical</type> -->
+            <type>custom</type>
+            <custom_function>
+              <c1>0.5</c1>
+              <c2>4.0</c2>
+              <f>1.0</f>
+              <fun>cos</fun>
+            </custom_function>
+            <scale_to_hfov>true</scale_to_hfov>
+            <cutoff_angle>3.14</cutoff_angle>
+            <env_texture_size>512</env_texture_size>
+          </lens>
+        </camera>
+        <plugin name="camera_controller" filename="libgazebo_ros_camera.so">
         <alwaysOn>true</alwaysOn>
-        <updateRate>30.0</updateRate>
-        <cameraName>camera_center_left</cameraName>
-        <frameName>camera_rgb_optical_center_left_frame</frameName>
-        <imageTopicName>rgb/image_raw</imageTopicName>
+        <updateRate>10.0</updateRate>
+        <cameraName>camera</cameraName>
+        <frameName>camera_rgb_optical_front_frame</frameName>
+        <imageTopicName>rgb/image_raw_front</imageTopicName>
         <cameraInfoTopicName>rgb/camera_info</cameraInfoTopicName>
-        <hackBaseline>0.07</hackBaseline>
+        <CxPrime></CxPrime>
+        <Cx></Cx>
+        <Cy></Cy>
+        <focalLength></focalLength>
+        <hackBaseline>0.7</hackBaseline>
         <distortionK1>0.0</distortionK1>
         <distortionK2>0.0</distortionK2>
@@ -323,34 +211,44 @@
         <distortionT2>0.0</distortionT2>
       </plugin>
-    </sensor>
-  </gazebo>
-<!--link : https://www.raspberrypi.org/documentation/hardware/camera/-->
-  <gazebo reference="camera_rgb_center_right_frame">
-    <sensor type="camera" name="camera_center_right">
-      <always_on>true</always_on>
-      <visualize>$(arg camera_visual)</visualize>
-      <camera>
-          <!--120°-->
-          <horizontal_fov>2.09</horizontal_fov>
+      </sensor>
+  </gazebo>
+  <gazebo reference="omnidirectional_camera_back_frame">
+      <sensor type="wideanglecamera" name="camera">
+        <camera>
+          <horizontal_fov>3.14</horizontal_fov>
           <image>
-              <!-- <width>694</width>
-              <height>520</height> -->
-              <width>640</width>
-              <height>480</height>
-              <format>R8G8B8</format>
+            <width>640</width>
+            <height>640</height>
           </image>
           <clip>
-              <near>0.03</near>
-              <far>100</far>
+            <near>0.1</near>
+            <far>50</far>
           </clip>
-      </camera>
-      <plugin name="camera_controller" filename="libgazebo_ros_camera.so">
+          <lens>
+            <!-- <type>gnomonical</type> -->
+            <type>custom</type>
+            <custom_function>
+              <c1>0.5</c1>
+              <c2>4.0</c2>
+              <f>1.0</f>
+              <fun>cos</fun>
+            </custom_function>
+            <scale_to_hfov>true</scale_to_hfov>
+            <cutoff_angle>3.14</cutoff_angle>
+            <env_texture_size>512</env_texture_size>
+          </lens>
+        </camera>
+        <plugin name="camera_controller" filename="libgazebo_ros_camera.so">
         <alwaysOn>true</alwaysOn>
-        <updateRate>30.0</updateRate>
-        <cameraName>camera_center_right</cameraName>
-        <frameName>camera_rgb_optical_center_right_frame</frameName>
-        <imageTopicName>rgb/image_raw</imageTopicName>
+        <updateRate>10.0</updateRate>
+        <cameraName>camera</cameraName>
+        <frameName>camera_rgb_optical_back_frame</frameName>
+        <imageTopicName>rgb/image_raw_back</imageTopicName>
         <cameraInfoTopicName>rgb/camera_info</cameraInfoTopicName>
-        <hackBaseline>0.07</hackBaseline>
+        <CxPrime></CxPrime>
+        <Cx></Cx>
+        <Cy></Cy>
+        <focalLength></focalLength>
+        <hackBaseline>0.7</hackBaseline>
         <distortionK1>0.0</distortionK1>
         <distortionK2>0.0</distortionK2>
@@ -359,128 +257,5 @@
         <distortionT2>0.0</distortionT2>
       </plugin>
-    </sensor>
-  </gazebo>
-<!--link : https://www.raspberrypi.org/documentation/hardware/camera/-->
-  <gazebo reference="camera_rgb_right_frame">
-    <sensor type="camera" name="camera_right">
-      <always_on>true</always_on>
-      <visualize>$(arg camera_visual)</visualize>
-      <camera>
-          <!--120°-->
-          <horizontal_fov>2.09</horizontal_fov>
-          <!--130°-->
-          <!-- <horizontal_fov>2.27</horizontal_fov> -->
-          <!--150°-->
-          <!-- <horizontal_fov>2.62</horizontal_fov> -->
-          <image>
-              <!-- <width>694</width> -->
-              <!-- <height>520</height> -->
-              <width>640</width>
-              <height>480</height>
-              <format>R8G8B8</format>
-          </image>
-          <clip>
-              <near>0.03</near>
-              <far>100</far>
-          </clip>
-      </camera>
-      <plugin name="camera_controller" filename="libgazebo_ros_camera.so">
-        <topicName>camera_right</topicName>
-        <alwaysOn>true</alwaysOn>
-        <updateRate>30.0</updateRate>
-        <cameraName>camera_right</cameraName>
-        <frameName>camera_rgb_optical_right_frame</frameName>
-        <imageTopicName>rgb/image_raw</imageTopicName>
-        <cameraInfoTopicName>rgb/camera_info</cameraInfoTopicName>
-        <hackBaseline>0.07</hackBaseline>
-        <distortionK1>0.0</distortionK1>
-        <distortionK2>0.0</distortionK2>
-        <distortionK3>0.0</distortionK3>
-        <distortionT1>0.0</distortionT1>
-        <distortionT2>0.0</distortionT2>
-      </plugin>
-    </sensor>
-  </gazebo>
-<!--link : https://www.raspberrypi.org/documentation/hardware/camera/-->
-  <gazebo reference="camera_rgb_right_left_frame">
-    <sensor type="camera" name="camera_right_left">
-      <always_on>true</always_on>
-      <visualize>$(arg camera_visual)</visualize>
-      <camera>
-          <!--120°-->
-          <horizontal_fov>2.09</horizontal_fov>
-          <image>
-              <!-- <width>694</width>
-              <height>520</height> -->
-              <width>640</width>
-              <height>480</height>
-              <format>R8G8B8</format>
-          </image>
-          <clip>
-              <near>0.03</near>
-              <far>100</far>
-          </clip>
-      </camera>
-      <plugin name="camera_controller" filename="libgazebo_ros_camera.so">
-        <topicName>camera_right_left</topicName>
-        <alwaysOn>true</alwaysOn>
-        <updateRate>30.0</updateRate>
-        <cameraName>camera_right_left</cameraName>
-        <frameName>camera_rgb_optical_right_left_frame</frameName>
-        <imageTopicName>rgb/image_raw</imageTopicName>
-        <cameraInfoTopicName>rgb/camera_info</cameraInfoTopicName>
-        <hackBaseline>0.07</hackBaseline>
-        <distortionK1>0.0</distortionK1>
-        <distortionK2>0.0</distortionK2>
-        <distortionK3>0.0</distortionK3>
-        <distortionT1>0.0</distortionT1>
-        <distortionT2>0.0</distortionT2>
-      </plugin>
-    </sensor>
-  </gazebo>
-<!--link : https://www.raspberrypi.org/documentation/hardware/camera/-->
-  <gazebo reference="camera_rgb_right_right_frame">
-    <sensor type="camera" name="camera_right_right">
-      <always_on>true</always_on>
-      <visualize>$(arg camera_visual)</visualize>
-      <camera>
-          <!--120°-->
-          <horizontal_fov>2.09</horizontal_fov>
-          <image>
-              <!-- <width>694</width>
-              <height>520</height> -->
-              <width>640</width>
-              <height>480</height>
-              <format>R8G8B8</format>
-          </image>
-          <clip>
-              <near>0.03</near>
-              <far>100</far>
-          </clip>
-      </camera>
-      <plugin name="camera_controller" filename="libgazebo_ros_camera.so">
-        <topicName>camera_right_right</topicName>
-        <alwaysOn>true</alwaysOn>
-        <updateRate>30.0</updateRate>
-        <cameraName>camera_right_right</cameraName>
-        <frameName>camera_rgb_optical_right_right_frame</frameName>
-        <imageTopicName>rgb/image_raw</imageTopicName>
-        <cameraInfoTopicName>rgb/camera_info</cameraInfoTopicName>
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
File: turtlebot3_description/urdf/turtlebot3_waffle_pi.urdf.xacro (robot description, xacro)
@@ -160,6 +160,6 @@
     </inertial>
   </link>
-  <joint name="camera_joint" type="fixed">
-    <origin xyz="0.073 -0.011 0.384" rpy="0 0.524 0"/>
+  <!-- <joint name="camera_joint" type="fixed">
+    <origin xyz="0.073 -0.011 0.084" rpy="0 0 0"/>
     <parent link="base_link"/>
     <child link="camera_link"/>
@@ -173,5 +173,4 @@
     </collision>
   </link>
-<!--center-->
   <joint name="camera_rgb_joint" type="fixed">
     <origin xyz="0.003 0.011 0.009" rpy="0 0 0"/>
@@ -185,110 +184,41 @@
     <child link="camera_rgb_optical_frame"/>
   </joint>
-  <link name="camera_rgb_optical_frame"/>
-<!--center_left-->
-  <joint name="camera_rgb_center_left_joint" type="fixed">
-    <origin xyz="0.003 0.011 0.009" rpy="0 0 0.088"/>
+  <link name="camera_rgb_optical_frame"/> -->
+  <joint name="camera_joint" type="fixed">
+    <origin xyz="0 0 0.6" rpy="0 0 0"/>
+    <parent link="base_link"/>
+    <child link="camera_link"/>
+  </joint>
+  <link name="camera_link">
+    <collision>
+      <origin xyz="0 0 0" rpy="0 0 0"/>
+      <geometry>
+        <box size="0.015 0.030 0.027"/>
+      </geometry>
+    </collision>
+  </link>
+  <joint name="camera_rgb_front_joint" type="fixed">
+    <origin xyz="0 0 0" rpy="1.57 0 0"/>
     <parent link="camera_link"/>
-    <child link="camera_rgb_center_left_frame"/>
-  </joint>
-  <link name="camera_rgb_center_left_frame"/>
-  <joint name="camera_rgb_optical_center_left_joint" type="fixed">
-    <origin xyz="0 0 0" rpy="-1.57 0 -1.57"/>
-    <parent link="camera_rgb_center_left_frame"/>
-    <child link="camera_rgb_optical_center_left_frame"/>
-  </joint>
-  <link name="camera_rgb_optical_center_left_frame"/>
-<!--center_right-->
-  <joint name="camera_rgb_center_right_joint" type="fixed">
-    <origin xyz="0.003 0.011 0.009" rpy="0 0 -0.088"/>
+    <child link="omnidirectional_camera_front_frame"/>
+  </joint>
+  <link name="omnidirectional_camera_front_frame"/>
+  <joint name="camera_rgb_optical_front_joint" type="fixed">
+    <origin xyz="0 0 0" rpy="0 0 0"/>
+    <parent link="omnidirectional_camera_front_frame"/>
+    <child link="camera_rgb_optical_front_frame"/>
+  </joint>
+  <link name="camera_rgb_optical_front_frame"/>
+  <joint name="camera_rgb_back_joint" type="fixed">
+    <origin xyz="0 0 0" rpy="-1.57 0 3.14"/>
     <parent link="camera_link"/>
-    <child link="camera_rgb_center_right_frame"/>
-  </joint>
-  <link name="camera_rgb_center_right_frame"/>
-  <joint name="camera_rgb_optical_center_right_joint" type="fixed">
-    <origin xyz="0 0 0" rpy="-1.57 0 -1.57"/>
-    <parent link="camera_rgb_center_right_frame"/>
-    <child link="camera_rgb_optical_center_right_frame"/>
-  </joint>
-  <link name="camera_rgb_optical_center_right_frame"/>
-<!--left-->
-  <joint name="camera_rgb_left_joint" type="fixed">
-    <!-- <origin xyz="0.003 0.111 0.009" rpy="0 0 0.175"/> -->
-     <origin xyz="0.003 0.211 0.009" rpy="0 0 0"/>
-    <parent link="camera_link"/>
-    <child link="camera_rgb_left_frame"/>
-  </joint>
-  <link name="camera_rgb_left_frame"/>
-  <joint name="camera_rgb_optical_left_joint" type="fixed">
-    <origin xyz="0 0 0" rpy="-1.57 0 -1.57"/>
-    <parent link="camera_rgb_left_frame"/>
-    <child link="camera_rgb_optical_left_frame"/>
-  </joint>
-  <link name="camera_rgb_optical_left_frame"/>
-<!--left_left-->
-  <joint name="camera_rgb_left_left_joint" type="fixed">
-     <origin xyz="0.003 0.211 0.009" rpy="0 0 0.088"/>
-    <parent link="camera_link"/>
-    <child link="camera_rgb_left_left_frame"/>
-  </joint>
-  <link name="camera_rgb_left_left_frame"/>
-  <joint name="camera_rgb_optical_left_left_joint" type="fixed">
-    <origin xyz="0 0 0" rpy="-1.57 0 -1.57"/>
-    <parent link="camera_rgb_left_left_frame"/>
-    <child link="camera_rgb_optical_left_left_frame"/>
-  </joint>
-  <link name="camera_rgb_optical_left_left_frame"/>
-<!--left_right-->
-  <joint name="camera_rgb_left_right_joint" type="fixed">
-     <origin xyz="0.003 0.211 0.009" rpy="0 0 -0.088"/>
-    <parent link="camera_link"/>
-    <child link="camera_rgb_left_right_frame"/>
-  </joint>
-  <link name="camera_rgb_left_right_frame"/>
-  <joint name="camera_rgb_optical_left_right_joint" type="fixed">
-    <origin xyz="0 0 0" rpy="-1.57 0 -1.57"/>
-    <parent link="camera_rgb_left_right_frame"/>
-    <child link="camera_rgb_optical_left_right_frame"/>
-  </joint>
-  <link name="camera_rgb_optical_left_right_frame"/>
-<!--right-->
-  <joint name="camera_rgb_right_joint" type="fixed">
-    <!-- <origin xyz="0.003 -0.089 0.009" rpy="0 0 -0.175"/> -->
-    <origin xyz="0.003 -0.189 0.009" rpy="0 0 0"/>
-    <parent link="camera_link"/>
-    <child link="camera_rgb_right_frame"/>
-  </joint>
-  <link name="camera_rgb_right_frame"/>
-  <joint name="camera_rgb_optical_right_joint" type="fixed">
-    <origin xyz="0 0 0" rpy="-1.57 0 -1.57"/>
-    <parent link="camera_rgb_right_frame"/>
-    <child link="camera_rgb_optical_right_frame"/>
-  </joint>
-  <link name="camera_rgb_optical_right_frame"/>
-<!--right_left-->
-  <joint name="camera_rgb_right_left_joint" type="fixed">
-    <origin xyz="0.003 -0.189 0.009" rpy="0 0 0.088"/>
-    <parent link="camera_link"/>
-    <child link="camera_rgb_right_left_frame"/>
-  </joint>
-  <link name="camera_rgb_right_left_frame"/>
-  <joint name="camera_rgb_optical_right_left_joint" type="fixed">
-    <origin xyz="0 0 0" rpy="-1.57 0 -1.57"/>
-    <parent link="camera_rgb_right_left_frame"/>
-    <child link="camera_rgb_optical_right_left_frame"/>
-  </joint>
-  <link name="camera_rgb_optical_right_left_frame"/>
-<!--right_right-->
-  <joint name="camera_rgb_right_right_joint" type="fixed">
-    <origin xyz="0.003 -0.189 0.009" rpy="0 0 -0.088"/>
-    <parent link="camera_link"/>
-    <child link="camera_rgb_right_right_frame"/>
-  </joint>
-  <link name="camera_rgb_right_right_frame"/>
-  <joint name="camera_rgb_optical_right_right_joint" type="fixed">
-    <origin xyz="0 0 0" rpy="-1.57 0 -1.57"/>
-    <parent link="camera_rgb_right_right_frame"/>
-    <child link="camera_rgb_optical_right_right_frame"/>
-  </joint>
-  <link name="camera_rgb_optical_right_right_frame"/>
+    <child link="omnidirectional_camera_back_frame"/>
+  </joint>
+  <link name="omnidirectional_camera_back_frame"/>
+  <joint name="camera_rgb_optical_back_joint" type="fixed">
+    <origin xyz="0 0 0" rpy="0 0 0"/>
+    <parent link="omnidirectional_camera_back_frame"/>
+    <child link="camera_rgb_optical_back_frame"/>
+  </joint>
+  <link name="camera_rgb_optical_back_frame"/>
 </robot>

Commit message: change urdf

File: turtlebot3_description/urdf/turtlebot3_waffle_pi.gazebo.xacro (robot description, xacro)
@@ -174,4 +174,6 @@
             <width>640</width>
             <height>640</height>
+            <!-- <width>694</width>
+            <height>520</height> -->
           </image>
           <clip>

File: turtlebot3_description/urdf/turtlebot3_waffle_pi.urdf.xacro (robot description, xacro)
@@ -187,4 +187,5 @@
   <joint name="camera_joint" type="fixed">
     <origin xyz="0 0 0.6" rpy="0 0 0"/>
+    <!-- <origin xyz="0.073 -0.011 0.384" rpy="0 0.524 0"/> -->
     <parent link="base_link"/>
     <child link="camera_link"/>
@@ -193,4 +194,5 @@
     <collision>
       <origin xyz="0 0 0" rpy="0 0 0"/>
+      <!-- <origin xyz="0.005 0.011 0.013" rpy="0 0 0"/> -->
       <geometry>
         <box size="0.015 0.030 0.027"/>
@@ -200,4 +202,5 @@
   <joint name="camera_rgb_front_joint" type="fixed">
     <origin xyz="0 0 0" rpy="1.57 0 0"/>
+    <!-- <origin xyz="0.003 0.011 0.009" rpy="0 0 0"/> -->
     <parent link="camera_link"/>
     <child link="omnidirectional_camera_front_frame"/>
@@ -206,4 +209,5 @@
   <joint name="camera_rgb_optical_front_joint" type="fixed">
     <origin xyz="0 0 0" rpy="0 0 0"/>
+    <!-- <origin xyz="0 0 0" rpy="-1.57 0 -1.57"/> -->
     <parent link="omnidirectional_camera_front_frame"/>
     <child link="camera_rgb_optical_front_frame"/>
